Commit message: changed approach

File: V3/src/robbie_simulator/src/urdf/robbie.urdf (robot description, URDF)
Before this commit: robot robot_arm, 5 links, 4 joints
Links:
- link base_link: geometry visual box size=0.2 0.2 0.05
- link link1: geometry visual box size=0.1 0.1 0.5
- link link2: geometry visual box size=0.1 0.1 0.5
- link link3: geometry visual box size=0.1 0.1 0.5
- link link4: geometry visual box size=0.1 0.1 0.5
Joints:
- joint joint1: limit lower=-3.14 upper=3.14 effort=100 velocity=1.0 -> lower=-3.14 upper=3.14 effort=1.0 velocity=1.0; origin xyz=0 0 0.1 rpy=0 0 0 -> xyz=0 0 0.05
- joint joint2: limit lower=-3.14 upper=3.14 effort=100 velocity=1.0 -> lower=-3.14 upper=3.14 effort=1.0 velocity=1.0; origin xyz=0 0 0.4 rpy=0 0 0 -> xyz=0 0 0.5
- joint joint3: limit lower=-3.14 upper=3.14 effort=100 velocity=1.0 -> lower=-3.14 upper=3.14 effort=1.0 velocity=1.0; origin xyz=0 0 0.4 rpy=0 0 0 -> xyz=0 0 0.5
- joint joint4: limit lower=-3.14 upper=3.14 effort=100 velocity=1.0 -> lower=-3.14 upper=3.14 effort=1.0 velocity=1.0; origin xyz=0 0 0.4 rpy=0 0 0 -> xyz=0 0 0.5
